File: Electronics/FED3_v6.3.sch (EAGLE design)
At the start: 50 parts, among them IC1 RTC_PCF8523T, IC2 TB6612 SSOP, IC3 M74VHC1GT50DTT1G, Q1 32.768, Q2 DMG3415, Q3 MOSFET_P-CH, SW1 SSSS811101

Commit message: Added a secondary connector to plug the battery.
Parts:
- added X1: B2B-PH-K-S(LF)(SN), Rembrandt Electronics - JST XH Connectors v1-0:JST-XH-02-PIN-ROUND-PAD
Connections:
- net GND: now also X1-1.S
- net VCC: now also X1-2.S
Other:
- note added: "Licensed under the TAPR Open Hardware License (www.tapr.org/OHL) Copyright 2019-2021 Mohamed Ali, FIlipe Carvalho, Alexxai Kravitz"
- note removed: "Licensed under the TAPR Open Hardware License (www.tapr.org/OHL) Copyright 2019 Mohamed Ali, FIlipe Carvalho, Alexxai Kravitz"
