File: Electronics/FED3_v7.1.sch (EAGLE design)
At the start: 51 parts, among them IC1 RTC_PCF8523T, IC2 TB6612 SSOP, IC3 M74VHC1GT50DTT1G, Q1 32.768, Q2 DMG3415, Q3 MOSFET_P-CH, SW1 SSSS811101, X1 B2B-PH-K-S(LF)(SN)

Commit message: Added two extra RGBs, replaced the BNC with an audio socket, and updated the license.
Parts:
- removed BNC: BNC, CNP-connectors:BNC
- removed ON: (no value), led:LEDCHIPLED_0603
- removed R10: 1k3, SparkFun:RESISTOR
- added C10, C9: 10uF, microbuilder:CAP_CERAMIC0805-NOOUTLINE
- added EXT: STEREO_JACK, CNP-connectors:STEREO_JACK
- added LED10, LED9: WS2812B5050, microbuilder:WS2812B5050
Connections:
- removed net N$8: ON.A, R10.1
- new net N$17: LED10.DI, LED9.DO
- new net N$18: LED8.DO, LED9.DI
- net 3V3: no longer R10.2
- net A0: now also EXT.4; no longer BNC.1
- net GND: now also C10.2, C9.2, EXT.5; no longer BNC.2, ON.C
- net VCCNEO: now also C10.1, C9.1, LED10.VDD, LED9.VDD
Other:
- note removed: "Licensed under the TAPR Open Hardware License (www.tapr.org/OHL) Copyright 2019-2021 Mohamed Ali, FIlipe Carvalho, Alexxai Kravitz"
- moved on the sheet: C5, C6, C7, C8, FEATHER_L, FEATHER_R, R12, X1-1, X1-2
