File: Electronics/old_PCB_designs/v5.2 (for use with Adafruit breakouts)/FED3_041319.sch (EAGLE design)
At the start: 19 parts, among them U1 GP1A57HR, U3 GP1A57HR, U4 GP1A57HR, X1 1-227161-0

Commit message: updated v5.2 PCB
Parts:
- renumbered I2C to AUX_I2C
Changed lines of the file:
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@@
 <?xml version="1.0" encoding="utf-8"?>
 <!DOCTYPE eagle SYSTEM "eagle.dtd">
-<eagle version="9.6.2">
+<eagle version="9.3.0">
 <drawing>
 <settings>
@@
 <part name="RTC" library="pinhead" deviceset="PINHD-1X5" device=""/>
 <part name="X1" library="con-coax" deviceset="?227161*" device="1-" technology="-0"/>
-<part name="I2C" library="pinhead" deviceset="PINHD-1X4" device=""/>
+<part name="AUX_I2C" library="pinhead" deviceset="PINHD-1X4" device=""/>
 </parts>
 <sheets>
@@
 <attribute name="NAME" x="96.52" y="59.182" size="1.778" layer="95"/>
 </instance>
-<instance part="I2C" gate="A" x="30.48" y="17.78" smashed="yes">
+<instance part="AUX_I2C" gate="A" x="30.48" y="17.78" smashed="yes">
 <attribute name="NAME" x="24.13" y="26.035" size="1.778" layer="95"/>
 <attribute name="VALUE" x="24.13" y="10.16" size="1.778" layer="96"/>
@@
 </segment>
 <segment>
-<pinref part="I2C" gate="A" pin="4"/>
+<pinref part="AUX_I2C" gate="A" pin="4"/>
 <wire x1="27.94" y1="15.24" x2="12.7" y2="15.24" width="0.1524" layer="91"/>
 <label x="12.7" y="15.24" size="1.778" layer="95"/>
@@
 </segment>
 <segment>
-<pinref part="I2C" gate="A" pin="1"/>
+<pinref part="AUX_I2C" gate="A" pin="1"/>
 <wire x1="27.94" y1="22.86" x2="12.7" y2="22.86" width="0.1524" layer="91"/>
 <label x="12.7" y="22.86" size="1.778" layer="95"/>
@@
 <wire x1="27.94" y1="17.78" x2="12.7" y2="17.78" width="0.1524" layer="91"/>
 <label x="12.7" y="17.78" size="1.778" layer="95"/>
-<pinref part="I2C" gate="A" pin="3"/>
+<pinref part="AUX_I2C" gate="A" pin="3"/>
 </segment>
 <segment>
@@
 <wire x1="27.94" y1="20.32" x2="12.7" y2="20.32" width="0.1524" layer="91"/>
 <label x="12.7" y="20.32" size="1.778" layer="95"/>
-<pinref part="I2C" gate="A" pin="2"/>
-</segment>
-<segment>
+<pinref part="AUX_I2C" gate="A" pin="2"/>
+</segment>
+<segment>
