File: Electronics/v7.3/IOs Interface.kicad_sch (KiCad schematic)
At the start: 28 parts, among them IC1 MC74VHC1GT125DBVT1G, Q2 DMP2035U-7

Commit message: Fixd some MPN and regenerated the BOM.
Parts:
- LED1, LED10, LED2, LED3, LED4, LED5, LED6, LED7, LED8, LED9: MPN SK6812RGBW-BW -> XT1511RGBW-BW
Changed lines of the file:
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@@
 			)
 		)
-		(property "MPN" "SK6812RGBW-BW"
+		(property "MPN" "XT1511RGBW-BW"
 			(at 187.96 74.93 0)
 			(effects
@@
 			)
 		)
-		(property "MPN" "SK6812RGBW-BW"
+		(property "MPN" "XT1511RGBW-BW"
 			(at 264.16 74.93 0)
 			(effects
@@
 			)
 		)
-		(property "MPN" "SK6812RGBW-BW"
+		(property "MPN" "XT1511RGBW-BW"
 			(at 238.76 74.93 0)
 			(effects
@@
 			)
 		)
-		(property "MPN" "SK6812RGBW-BW"
+		(property "MPN" "XT1511RGBW-BW"
 			(at 86.36 74.93 0)
 			(effects
@@
 			)
 		)
-		(property "MPN" "SK6812RGBW-BW"
+		(property "MPN" "XT1511RGBW-BW"
 			(at 238.76 114.3 0)
 			(effects
@@
 			)
 		)
-		(property "MPN" "SK6812RGBW-BW"
+		(property "MPN" "XT1511RGBW-BW"
 			(at 137.16 74.93 0)
 			(effects
@@
 			)
 		)
-		(property "MPN" "SK6812RGBW-BW"
+		(property "MPN" "XT1511RGBW-BW"
 			(at 111.76 74.93 0)
 			(effects
@@
 			)
 		)
-		(property "MPN" "SK6812RGBW-BW"
+		(property "MPN" "XT1511RGBW-BW"
 			(at 264.16 114.3 0)
 			(effects
@@
 			)
 		)
-		(property "MPN" "SK6812RGBW-BW"
+		(property "MPN" "XT1511RGBW-BW"
 			(at 162.56 74.93 0)
 			(effects
@@
 			)
 		)
-		(property "MPN" "SK6812RGBW-BW"
+		(property "MPN" "XT1511RGBW-BW"
 			(at 213.36 74.93 0)
 			(effects
