File: Electronics/v7.3/FED3_v7.3.kicad_sch (KiCad schematic)
At the start: 26 parts, among them IC2 TB6612FNG, SW1 Sw, U2 SPX3819-3.3, U3 MCP73831T, X5 JST-XH-02

Commit message: Replaced RED LED because it's obsolete.
Parts:
- CHG0, L2: MPN 5975004407F -> VFHR1116P-4C82A-TR; OEPSPN OEPS030006 -> OEPS030038
Changed lines of the file:
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@@
 			)
 		)
-		(property "OEPSPN" "OEPS030006"
+		(property "OEPSPN" "OEPS030038"
 			(at 113.03 92.71 0)
 			(effects
@@
 			)
 		)
-		(property "MPN" "5975004407F"
+		(property "MPN" "VFHR1116P-4C82A-TR"
 			(at 113.03 92.71 0)
 			(effects
@@
 			)
 		)
-		(property "OEPSPN" "OEPS030006"
+		(property "OEPSPN" "OEPS030038"
 			(at 171.45 40.005 0)
 			(effects
@@
 			)
 		)
-		(property "MPN" "5975004407F"
+		(property "MPN" "VFHR1116P-4C82A-TR"
 			(at 171.45 40.005 0)
 			(effects
