File: Electronics/v7.4/FED3.kicad_sch (KiCad schematic)
At the start: 29 parts, among them IC2 TB6612FNG, SW1 Sw, U2 MIC5504-3.3, U3 MCP73831T, X5 JST-XH-02

Commit message: Decreased consumption and added STEMMA connector.
- Updated Bat's resistor divider to 0.1% tolerance
- Reduced LEDs' current to bellow 1 mA
- Updated buzzer model
- Increased available voltage to motor
- Added STEMMA (2mm ) connector

To do:
- Update STEMMA to STEMMA QT (2mm)
- (Maybe) Update charging current to slightly bellow 500 mA

Co-Authored-By: David Palma <78764277+davidpalma666@users.noreply.github.com>
Parts:
- removed D2: SM5817PL, Diode_SMD:D_SOD-123F, symbol FED3 SymbLib:DIODE-SCHOTTKYSOD-123
- L2: value RED -> DNP; MPN 5975004407F -> n.a.; OEPSPN OEPS030006 -> n.a.; now not fitted; now left out of the parts list
- R11, R16, R17: value 100k -> 100k 0.1%; MPN ERJ-2RKF1003X -> RG1005P-104-B-T5; OEPSPN OEPS020019 -> OEPS020175
- R19: value 68R -> DNP; MPN RCS040268R0FKED -> n.a.; OEPSPN OEPS020032 -> n.a.; now not fitted; now left out of the parts list
- R7: now not fitted; now left out of the parts list
- TP5: now left out of the parts list
Connections:
- net VBat: now also C11.1, C4.1, IC2.13 (VM@2), IC2.14 (VM@3), IC2.24 (VM@1), R11.1, U2.1 (IN)
- net VUSB: no longer C11.1, C4.1, IC2.13 (VM@2), IC2.14 (VM@3), IC2.24 (VM@1), R11.1, U2.1 (IN)

Commit message: Updated supply circuit, battery charge current, and added a new connector.
- Added a STEMMA QT / Qwiic connector for expansion.
- Made the entire supply being sourced from the battery.
- Reduced battery charging to 455 mA (previously was 500 mA).

Co-Authored-By: David Palma <78764277+davidpalma666@users.noreply.github.com>
Parts:
- removed R20: 1k, Resistor_SMD:R_0402_1005Metric, symbol Device:R_US
- R14: value 1k -> 2k2; MPN ERJ-2RKF1001X -> ERJ-2RKF2201X; OEPSPN OEPS020006 -> OEPS020174
Connections:
- net GND: now also R14.1
Other:
- note added: "2.2K = 455mA"
Changed lines of the file:
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@@
 	(text "5.0K  = 200mA"
 		(exclude_from_sim no)
-		(at 207.645 34.29 0)
+		(at 207.772 32.385 0)
 		(effects
 			(font
@@
 		)
 	)
+	(text "2.2K  = 455mA"
+		(exclude_from_sim no)
+		(at 207.772 34.29 0)
+		(effects
+			(font
+				(size 1.2 1.2)
+			)
+			(justify left bottom)
+		)
+	)
 	(text "1.0K  = 1000mA"
 		(exclude_from_sim no)
@@
 	(text "10K  = 100mA"
 		(exclude_from_sim no)
-		(at 207.645 32.385 0)
+		(at 207.772 30.48 0)
 		(effects
 			(font
@@
 	(wire
 		(pts
-			(xy 222.25 44.45) (xy 222.25 43.18)
+			(xy 222.25 43.18) (xy 222.25 53.34)
 		)
 		(stroke
@@
 	(wire
 		(pts
-			(xy 222.25 52.07) (xy 222.25 53.34)
-		)
-		(stroke
-			(width 0)
-			(type solid)
-		)
-	)
-	(wire
-		(pts
 			(xy 224.79 134.62) (xy 227.33 134.62)
 		)
@@
 			)
 		)
-		(property "Value" "1k"
+		(property "Value" "2k2"
 			(at 211.582 48.006 90)
 			(effects
@@
 			)
 		)
-		(property "Description" "SMD 0402 1kΩ ±1% 0.100W"
+		(property "Description" "SMD 0402 2.2kΩ ±1% 0.100W"
 			(at 213.36 43.18 0)
 			(effects
@@
 			)
 		)
-		(property "OEPSPN" "OEPS020006"
+		(property "OEPSPN" "OEPS020174"
 			(at 213.36 43.18 0)
 			(effects
@@
 			)
 		)
-		(property "MPN" "ERJ-2RKF1001X"
+		(property "MPN" "ERJ-2RKF2201X"
 			(at 213.36 43.18 0)
 			(effects
@@
 					(unit 1)
 				)
-			)
-		)
-	)
-	(symbol
-		(lib_id "Device:R_US")
-		(at 222.25 48.26 0)
-		(mirror x)
-		(unit 1)
-		(exclude_from_sim no)
-		(in_bom yes)
-		(on_board yes)
-		(dnp no)
-		(property "Reference" "R20"
-			(at 220.726 47.498 0)
-			(effects
-				(font
-					(size 1.27 1.27)
-				)
-				(justify right)
-			)
-		)
-		(property "Value" "1k"
-			(at 220.726 50.038 0)
-			(effects
-				(font
-					(size 1.27 1.27)
-				)
-				(justify right)
-			)
-		)
-		(property "Footprint" "Resistor_SMD:R_0402_1005Metric"
-			(at 222.25 48.26 0)
-			(effects
-				(font
-					(size 1.27 1.27)
-				)
-				(hide yes)
-			)
-		)
-		(property "Datasheet" ""
-			(at 222.25 48.26 0)
-			(effects
-				(font
-					(size 1.27 1.27)
-				)
-				(hide yes)
-			)
-		)
-		(property "Description" "SMD 0402 1kΩ ±1% 0.100W"
-			(at 222.25 48.26 0)
-			(effects
-				(font
-					(size 1.27 1.27)
-				)
-				(hide yes)
-			)
-		)
-		(property "OEPSPN" "OEPS020006"
-			(at 222.25 48.26 0)
-			(effects
-				(font
-					(size 1.27 1.27)
-				)
-				(hide yes)
-			)
-		)
-		(property "MPN" "ERJ-2RKF1001X"
-			(at 222.25 48.26 0)
-			(effects
-				(font
-					(size 1.27 1.27)
-				)
-				(hide yes)
-			)
-		)
-		(pin "1"
-		)
-		(pin "2"
-		)
-		(instances
-			(project "FED3_v7.3"
-				(path "/2ba63f12-2fcd-4471-9636-2762cde37de8"
-					(reference "R20")
-					(unit 1)
-				)

Commit message: Added schematic sheet
- Fixed some typos
Other:
- sheet controler stage renamed Controller Stage
- company: (none) -> Kravitz Lab
- title: (none) -> FED3 Control Board
Changed lines of the file:
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@@
 	(generator_version "9.0")
 	(paper "A4")
+	(title_block
+		(title "FED3 Control Board")
+		(rev "7.4")
+		(company "Kravitz Lab")
+		(comment 1 "Open Ephys, Inc.")
+	)
 	(rectangle
 		(start 161.29 14.605)
@@
 			(color 202 239 212 1.0000)
 		)
-		(property "Sheetname" "controler stage"
+		(property "Sheetname" "Controller Stage"
 			(at 26.67 139.1314 0)
 			(effects
@@
 	)
 	(embedded_fonts no)
+	(embedded_files
+		(file
+			(name "generic.kicad_wks")
+			(type worksheet)
+			(data |KLUv/WDdCX0VAPbdXiHwth4UjMf84wQpaKiddXNyw2vE3ASpJOKm/UZkMyvPewFVAE4AWAA71P+6
+				E/V/PHhP6hl7NhdyvnNBg6Vy+uc/TLoZgwYrqd8THr90vwAABASi6O845VVxKvxdDihWvvVz++br
+				MViUUkSd1bPG476jAiAgGEMkzsd5OFQI1UctVrTy7u1E2OrTmkrby9ifu+L1uW/e2nvQp88q5Gmw
+				8ws+fr+f9y+L9Oa88s83DLU3p1VMWf3Lt9ZppVX9shLSUuq/uR+rym/I5fdulhPePlB3nqiaJruM
+				7sWyKo9QmUhQSqlo2yXTcBxYQ4ugCHXaOS+p8GvKeqUyDObgZJlt01AEZ9znHHtv076fr+emDv5R
+				BLLVKWaq1mfXdZMiCoDPukPdBgGBofrisvaiijoRFEPJJqbMiaFuzLqhYJZJpTHlApNlkM2yEDIx
+				wSiZRHvgh4dB7rEbqteFnDSTYDQM+BhzSVrph/3v/WyDQ2rwaZU/F27d8X1FznLJLFiAhKDhRMcY
+				khEJkiRJOnBEpOSqG67IIUSIB6wVkypOj83iBj0zp4LL2kMMw+lEgMAIPplQr3guKCdlw/SfU9Pm
+				wv5Qjf2c0i+iukyGwJWg6H+jq3g9lh1bbaelmbDHUSOcHe0f4IqIU3pYnNopN2UGuqm6tUzbD0DL
+				A846XZ/tXUnW1CdqEKGhzI4PDvNZEWdNQVTqjKoxCJiOkLlyPnE2aN0Mgntwtl4Il0TKJW3CO+mz
+				Z3UY05BTT9QUnWnIY2O5jqbO0VBDfwAQ0J2lPShW8OIwbtD7c16HHQWSRlikdRdv3bO2EHlrLTcN
+				okDmqiZIAfyy8oU9FMxL3Rl0kbp+k4D31UmB0+QSWL73QeUaK7tJbNu8DHaE+JnfMeyjQJuerxNn
+				/RsMH2E/mWuAPwa9Cg==|
+			)
+			(checksum "29ED9DE70340A48902A32D9A43F096A1")
+		)
+	)
 )

Commit message: Prepared files for production.
Also fixed #13
Parts:
- IC2: MPN TB6612FNG,C,8,EL -> TB6612FNG,C,8,EL
- L2, MOTOR0, R19, R7: now in the parts list
- SW1: MPN SSSS811101 -> SSSS811101
Changed lines of the file:
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@@
 		(unit 1)
 		(exclude_from_sim no)
-		(in_bom no)
+		(in_bom yes)
 		(on_board yes)
 		(dnp yes)
@@
 			)
 		)
-		(property "MPN" "SSSS811101 "
+		(property "MPN" "SSSS811101"
 			(at 102.87 40.64 0)
 			(effects
@@
 		(unit 1)
 		(exclude_from_sim no)
-		(in_bom no)
+		(in_bom yes)
 		(on_board yes)
 		(dnp yes)
@@
 			)
 		)
-		(property "MPN" "TB6612FNG,C,8,EL "
+		(property "MPN" "TB6612FNG,C,8,EL"
 			(at 204.47 124.46 0)
 			(effects
@@
 		(unit 1)
 		(exclude_from_sim no)
-		(in_bom no)
+		(in_bom yes)
 		(on_board yes)
 		(dnp yes)
@@
 		(unit 1)
 		(exclude_from_sim no)
-		(in_bom no)
-		(on_board yes)
-		(dnp no)
+		(in_bom yes)
+		(on_board yes)
+		(dnp no)

Commit message: Replaced obsolete LED.
Parts:
- CHG0: MPN 5975004407F -> VFHR1116P-4C82A-TR; OEPSPN OEPS030006 -> OEPS030038
Changed lines of the file:
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@@
 			)
 		)
-		(property "OEPSPN" "OEPS030006"
+		(property "OEPSPN" "OEPS030038"
 			(at 171.45 40.005 0)
 			(effects
@@
 			)
 		)
-		(property "MPN" "5975004407F"
+		(property "MPN" "VFHR1116P-4C82A-TR"
 			(at 171.45 40.005 0)
 			(effects
