File: Electronics/v7.4/FED3.kicad_sch (KiCad schematic)
At the start: 27 parts, among them IC2 TB6612FNG, SW1 Sw, U2 MIC5504-3.3, U3 MCP73831T, X5 JST-XH-02

Commit message: Fixed bad MPN of the battery's connector.
Parts:
- X5: value JST-XH-02 -> B2B-PH-K-S; MPN B2B-XH-A(LF)(SN) -> B2B-PH-K-S(LF)(SN); OEPSPN OEPS070028 -> OEPS070130
Changed lines of the file:
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@@
 			)
 		)
-		(property "Value" "JST-XH-02"
+		(property "Value" "B2B-PH-K-S"
 			(at 83.82 49.53 0)
 			(effects
@@
 			)
 		)
-		(property "OEPSPN" "OEPS070028"
+		(property "OEPSPN" "OEPS070130"
 			(at 82.55 46.99 0)
 			(effects
@@
 			)
 		)
-		(property "MPN" "B2B-XH-A(LF)(SN)"
+		(property "MPN" "B2B-PH-K-S(LF)(SN)"
 			(at 82.55 46.99 0)
 			(effects
