File: Electronics/v7.4/FED3.kicad_pcb (KiCad board)
At the start: 4 copper layers, 108 x 50 mm, 89 parts, among them IC1 MC74VHC1GT125, IC2 TB6612FNG, IC4 RTC PCF8523T, J1 Conn_02x03_Odd_Even, Q2 DMP2035U-7, SW1 Sw, SW2 SPST_TACT-KMR2, U1 ATSAMD21G18A, U2 MIC5504-3.3, U3 MCP73831T, X1 ClockXtal, X2 uXtal, X4 microsd, X5 JST-XH-02

Commit message: Fixed bad MPN of the battery's connector.
Parts:
- X5: value JST-XH-02 -> B2B-PH-K-S
Changed lines of the file:
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@@
 			)
 		)
-		(property "Value" "JST-XH-02"
+		(property "Value" "B2B-PH-K-S"
 			(at -5.1 -1.3 0)
 			(unlocked yes)
@@
 			)
 		)
-		(property "OEPSPN" "OEPS070028"
+		(property "OEPSPN" "OEPS070130"
 			(at 0 0 180)
 			(unlocked yes)
@@
 			)
 		)
-		(property "MPN" "B2B-XH-A(LF)(SN)"
+		(property "MPN" "B2B-PH-K-S(LF)(SN)"
 			(at 0 0 180)
 			(unlocked yes)
@@
 			)
 		)
-		(property "Description" "DIODE: LED 0603 Red 635nm 20mA [VFHR1116P-4C82A-TR] [0603]"
+		(property "Description" "Light emitting diode"
 			(at 0 0 270)
 			(unlocked yes)
