File: Electronics/v7.5/FED3.kicad_pcb (KiCad board)
At the start: 4 copper layers, 108 x 50 mm, 96 parts, among them IC1 MC74VHC1GT125, IC2 TB6612FNG, IC4 RTC PCF8523T, J1 Conn_02x03_Odd_Even, J2 Conn_01x02_Odd_Even, J3 USB4105-GF-A, Q1 DMP2035U-7, SW1 Sw, SW2 SPST_TACT-KMR2, U1 ATSAMD21G18A, U2 MIC5504-3.3, U3 MCP73834-xxxx, X1 ClockXtal, X2 uXtal, X3 B2B-PH-K-S, X4 microsd

Commit message: Added MPN and OEPS PN to remaining components.
Parts:
- R18: value DNP -> 4k7
Changed lines of the file:
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@@
 			)
 		)
-		(property "OEPSPN" "_TBD"
+		(property "OEPSPN" "OEPS080177"
 			(at 0 0 180)
 			(unlocked yes)
@@
 			)
 		)
-		(property "MPN" "MCP73834-xxxx"
+		(property "MPN" "MCP73834-CNI/MF"
 			(at 0 0 180)
 			(unlocked yes)
@@
 			)
 		)
-		(property "Description" "SMD 0402 1kΩ ±1% 0.100W"
+		(property "Description" "SMD 0402 4k7"
 			(at 0 0 270)
 			(unlocked yes)
@@
 			)
 		)
-		(property "Value" "DNP"
+		(property "Value" "4k7"
 			(at 0 1.17 90)
 			(unlocked yes)
@@
 			)
 		)
-		(property "Description" ""
+		(property "Description" "SMD 0402 4k7"
 			(at 0 0 90)
 			(unlocked yes)
@@
 			)
 		)
-		(property "OEPSPN" "n.a."
+		(property "OEPSPN" "OEPS020010"
 			(at 0 0 90)
 			(unlocked yes)
@@
 			)
 		)
-		(property "MPN" "n.a."
+		(property "MPN" "ERJ-2RKF4701X"
 			(at 0 0 90)
 			(unlocked yes)
@@
 			)
 		)
-		(property "OEPSPN" "n.a."
+		(property "OEPSPN" "OEPS00000"
 			(at 0 0 90)
 			(unlocked yes)
@@
 		(sheetname "/")
 		(sheetfile "FED3.kicad_sch")
-		(attr smd)
+		(attr smd dnp)
 		(fp_line
 			(start -0.153641 -0.38)
@@
 			)
 		)
-		(property "OEPSPN" "n.a."
+		(property "OEPSPN" "OEPS070131"
 			(at 0 0 0)
 			(unlocked yes)
@@
 			)
 		)
-		(property "MPN" "n.a."
+		(property "MPN" "M20-9990546"
 			(at 0 0 0)
 			(unlocked yes)
@@
 			)
 		)
-		(property "OEPSPN" "n.a."
+		(property "OEPSPN" "OEPS00000"
 			(at 0 0 180)
 			(unlocked yes)
