File: Electronics/v7.6/IOs Interface.kicad_sch (KiCad schematic)
At the start: 30 parts, among them IC1 MC74VHC1GT125, Q1 DMP2035U-7

Commit message: Updated 330Ω resistor specs and part numbers
Updated the description, OEPSPN, and MPN for 330Ω SMD 0402 resistors in schematic and PCB files to reflect a new part (CRCW0402330RFKEDHP, 0.200W).
Parts:
- R12: MPN RC0402FR-07330RL -> CRCW0402330RFKEDHP; OEPSPN OEPS020037 -> OEPS020191
Changed lines of the file:
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@@
 			)
 		)
-		(property "Description" "SMD 0402 330Ω ±1% 0.063W"
+		(property "Description" "SMD 0402 330Ω ±1% 0.200W"
 			(at 67.31 77.47 0)
 			(effects
@@
 			)
 		)
-		(property "OEPSPN" "OEPS020037"
+		(property "OEPSPN" "OEPS020191"
 			(at 67.31 77.47 0)
 			(effects
@@
 			)
 		)
-		(property "MPN" "RC0402FR-07330RL"
+		(property "MPN" "CRCW0402330RFKEDHP"
 			(at 67.31 77.47 0)
 			(effects
