File: Electronics/v7.6/IOs Interface.kicad_sch (KiCad schematic)
At the start: 30 parts, among them IC1 MC74VHC1GT125, Q1 DMP2035U-7

Commit message: Replaced R26 with new value and footprint.
Removed the 0402 330Ω resistor R26 from the top layer and added a new 0805 510Ω resistor R26 on the bottom layer with updated MPN and OEPSPN. Changed back R12 to previous MPN and OEPS PN.
Parts:
- R12: MPN CRCW0402330RFKEDHP -> RC0402FR-07330RL; OEPSPN OEPS020191 -> OEPS020037
Changed lines of the file:
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@@
 			)
 		)
-		(property "Description" "SMD 0402 330Ω ±1% 0.200W"
+		(property "Description" "SMD 0402 330Ω ±1% 0.063W"
 			(at 67.31 77.47 0)
 			(effects
@@
 			)
 		)
-		(property "OEPSPN" "OEPS020191"
+		(property "OEPSPN" "OEPS020037"
 			(at 67.31 77.47 0)
 			(effects
@@
 			)
 		)
-		(property "MPN" "CRCW0402330RFKEDHP"
+		(property "MPN" "RC0402FR-07330RL"
 			(at 67.31 77.47 0)
 			(effects

Commit message: Add D2.0mm testpoints and PCB fixes
Parts:
- TP2: footprint TestPoint:TestPoint_Pad_1.0x1.0mm -> TestPoint:TestPoint_Pad_D2.0mm
Changed lines of the file:
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@@
 			)
 		)
-		(property "Footprint" "TestPoint:TestPoint_Pad_1.0x1.0mm"
+		(property "Footprint" "TestPoint:TestPoint_Pad_D2.0mm"
 			(at 115.57 26.67 0)
 			(effects
